File: 4runner-seat-heat-kicad/4runner-seat-heat.kicad_pcb (KiCad board)
At the start: 2 copper layers, 74.4 x 66.2 mm, 74 parts, among them J1 Toyota-90980-10964, J10 TE796864-3, J3 TE-284539-6, J4 TE-796859-2, J5 Toyota-90980-10933, J6 TE-796859-2, J7 TE-284510-6, J8 TE-284539-6, J9 TE-796859-3, Q1 BUK9Y30-75B,115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

Commit message: add moutning holes, export of Gerbers for rev02 and step files
Parts:
- removed 4runnerGraphic: G*****, _4runner-seat-heat-custom-libraries:4runner-logo-graphic
- removed 4runnerGraphic: G*****, _4runner-seat-heat-custom-libraries:4runner-front-graphic
- removed J10: TE796864-3, _4runner-seat-heat-custom-libraries:TE-796864-3
- removed the REF** at (58.3, 4.37)
- removed the REF** at (13.0, 4.37)
- removed the REF** at (58.5, 61.7)
- removed the REF** at (13.0, 61.7)
- added R21: 0ohm, Resistor_SMD:R_0603_1608Metric, F.Cu at (12.0, 29.7)
- added R22: 0ohm, Resistor_SMD:R_0603_1608Metric, F.Cu at (12.0, 31.5)
- added R23: 0ohm, Resistor_SMD:R_0603_1608Metric, F.Cu at (11.8, 49.2)
- added R24: 0ohm, Resistor_SMD:R_0603_1608Metric, F.Cu at (11.3, 43.8)
- added REF**: 4-40 Mount, _4runner-seat-heat-custom-libraries:4-40-Mounting-Hole, F.Cu at (13.3, 61.7)
- added REF**: 4-40 Mount, _4runner-seat-heat-custom-libraries:4-40-Mounting-Hole, F.Cu at (13.3, 0.71)
- added REF**: 4-40 Mount, _4runner-seat-heat-custom-libraries:4-40-Mounting-Hole, F.Cu at (58.5, 61.7)
- added REF**: 4-40 Mount, _4runner-seat-heat-custom-libraries:4-40-Mounting-Hole, F.Cu at (58.5, 0.71)
- J9: value TE-796859-3 -> TE-796866-4; footprint _4runner-seat-heat-custom-libraries:DNP-Mechanical -> _4runner-seat-heat-custom-libraries:TE-796864-4
- moved J9 53.9 mm to (64.3, 17.4), turned to 90 degrees
- moved J8 0.58 mm to (8.00, 38.0)
- moved J3 0.58 mm to (8.00, 6.41)
Connections:
- J3 pad 5: +12-Polyfuse -> DIMMER-GND
- J3 pad 6: Right-Illum -> Net-(J3-Pad6)
- J8 pad 5: +12-Polyfuse -> DIMMER-GND
- J8 pad 6: Left-Illum -> Net-(J8-Pad6)
- J9 pad 1: Net-(J9-Pad1) -> GND
- J9 pad 2: Net-(J9-Pad2) -> /12VDC-IGN
- J9 pad 3: Net-(J9-Pad3) -> +12-TAIL
- J9 pad 4: (no net) -> DIMMER-GND
- R19 pad 2: +Lights -> +12-TAIL
- U2 pad 11: Net-(U2-Pad11) -> Net-(R17-Pad1)
- U2 pad 17: Net-(R17-Pad1) -> Net-(U2-Pad17)
Routing:
- net +Lights: track 129.2 -> 0.00 mm
- net +12-TAIL: track 0.00 -> 128.4 mm, vias 0 -> 2
- net DIMMER-GND: track 0.00 -> 122.6 mm
- net Net-(R17-Pad1): track 24.3 -> 46.3 mm
- net Net-(J8-Pad6): track 0.00 -> 13.8 mm
- net +12-Polyfuse: track 86.4 -> 75.3 mm
- net Left-Illum: track 13.6 -> 2.65 mm
- net Net-(J3-Pad6): track 0.00 -> 8.84 mm
- net +12VDC: track 224.1 -> 218.7 mm, vias 0 -> 1
- net Right-Illum: track 5.25 -> 4.15 mm
- net Net-(J3-Pad2): track 6.02 -> 7.02 mm
- net GND: vias 259 -> 260
Other:
- board size 74.4 x 66.2 mm -> 74.4 x 71.5 mm
- board text added: "12V-TAIL"
- board text added: "12VDC IGN"
- board text added: "DIM-GND"
- board text added: "Heated Seat Interface ASL March 22 Rev02"
- board text added: "LeftHeat"
- board text added: "LeftIllum"
- board text added: "RightHeat"
- board text added: "RightIllum"
- board text added: "Teensy 3.1/3.2/LC"
- board text removed: "12VDC"
- board text removed: "Heated Seat Interface ASL Dec '21 Rev01.1"
- board text removed: "Lights"
