File: 4runner-seat-heat/4runner-seat-heat.sch (KiCad schematic (older format))
At the start: 70 parts, among them J1 Toyota-90980-10964, J10 TE796864-3, J2 TE-284510-6, J3 TE-284539-6, J4 TE-796859-2, J5 Toyota-90980-10933, J6 TE-796859-2, J7 TE-284510-6, J8 TE-284539-6, J9 TE-796859-3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

Commit message: refresh submodules
Parts:
- J10: symbol _4runner-seat-heat-custom-libraries:TE796864-3 -> 4runner-seat-heat-rescue:TE796864-3-_4runner-seat-heat-custom-libraries
Other:
- note added: "Pin: 6x TE-1743655-1"
Changed lines of the file:
@@
 	9235 7605 11045 7605
 $Comp
-L _4runner-seat-heat-custom-libraries:TE796864-3 J10
+L 4runner-seat-heat-rescue:TE796864-3-_4runner-seat-heat-custom-libraries J10
 U 1 1 61D4C3BB
 P 2995 5230
@@
 Text GLabel 10620 7705 2    50   Input ~ 0
 +Lights
+Text Notes 3150 2350 0    50   ~ 0
+Pin: 6x TE-1743655-1
+Text Notes 3150 4350 0    50   ~ 0
+Pin: 6x TE-1743655-1
 $EndSCHEMATC
